File: Ex1.kicad_pcb (KiCad board)
At the start: 2 copper layers, 154 parts, among them J1 Conn_01x02, J10 Conn_02x08_Odd_Even, J2 Conn_01x02, J4 Conn_01x08_Socket, J5 Conn_01x08_Socket, J6 Conn_01x08_Socket, J7 Conn_01x08_Socket, J8 Conn_01x04_Socket, J9 Conn_01x04_Socket, K1 G5NB, K2 G5NB, K3 G5NB, K4 G5NB, P1 Conn_02x03, Q1 C1815, Q10 7002_GSD, Q11 7002_GSD, Q12 7002_GSD, Q13 7002_GSD, Q14 7002_GSD, Q15 7002_GSD, Q16 7002_GSD, Q17 7002_GSD, Q2 C1815, Q3 C1815, Q4 C1815, Q5 C1815, Q6 7002_GSD, Q7 7002_GSD, Q8 7002_GSD, Q9 7002_GSD, SW3 RST, U1 LM2596S-ADJ, U2 XL1509-5.0, U3 PC817, U4 LM1117DT-3.3, U5 STM32F103CBTx, U6 PC817, U7 PC817, U8 PC817, Y1 8MHz, Y2 32.768K

Commit message: abc
Routing:
- net 0VDC: vias 29 -> 30
Other:
- board outline added: 125 x 75 mm
Changed lines of the file:
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@@
 			(drillshape 0)
 			(scaleselection 1)
-			(outputdirectory "../GERBER/")
+			(outputdirectory "Gerber/")
 		)
 	)
@@
 		(layer "Dwgs.User")
 	)
-	(gr_line
-		(start 64.5 37)
-		(end 189.5 37)
+	(gr_circle
+		(center 67.746365 108.695391)
+		(end 69.746365 108.695391)
 		(stroke
 			(width 0.2)
 			(type default)
 		)
+		(fill no)
 		(layer "Dwgs.User")
 	)
-	(gr_line
-		(start 189.5 112)
-		(end 64.5 112)
+	(gr_circle
+		(center 186.250676 108.695391)
+		(end 188.250676 108.695391)
 		(stroke
 			(width 0.2)
 			(type default)
 		)
+		(fill no)
 		(layer "Dwgs.User")
 	)
-	(gr_line
-		(start 64.5 112)
-		(end 64.5 37)
+	(gr_circle
+		(center 186.250676 40.296349)
+		(end 188.250676 40.296349)
 		(stroke
 			(width 0.2)
 			(type default)
 		)
+		(fill no)
 		(layer "Dwgs.User")
 	)
-	(gr_circle
-		(center 67.746365 108.695391)
-		(end 69.746365 108.695391)
+	(gr_line
+		(start 64.5 37)
+		(end 189.5 37)
 		(stroke
 			(width 0.2)
-			(type default)
+			(type solid)
 		)
-		(fill no)
-		(layer "Dwgs.User")
+		(layer "Edge.Cuts")
 	)
-	(gr_circle
-		(center 186.250676 108.695391)
-		(end 188.250676 108.695391)
+	(gr_line
+		(start 189.5 112)
+		(end 64.5 112)
 		(stroke
 			(width 0.2)
-			(type default)
+			(type solid)
 		)
-		(fill no)
-		(layer "Dwgs.User")
+		(layer "Edge.Cuts")
 	)
 	(gr_line
-		(start 189.5 37)
-		(end 189.5 112)
+		(start 64.5 112)
+		(end 64.5 37)
 		(stroke
 			(width 0.2)
-			(type default)
+			(type solid)
 		)
-		(layer "Dwgs.User")
+		(layer "Edge.Cuts")
 	)
-	(gr_circle
-		(center 186.250676 40.296349)
-		(end 188.250676 40.296349)
+	(gr_line
+		(start 189.5 37)
+		(end 189.5 112)
 		(stroke
 			(width 0.2)
-			(type default)
+			(type solid)
 		)
-		(fill no)
-		(layer "Dwgs.User")
+		(layer "Edge.Cuts")
 	)
 	(segment
@@
 		(net 5)
 	)
+	(via
+		(at 142.2 77.1)
+		(size 0.6)
+		(drill 0.3)
+		(layers "F.Cu" "B.Cu")
+		(free yes)
+		(net 5)
+	)
